Commit message: Great, now camera is working and available in rviz

File: src/vio/urdf/gazebo.xacro (robot description, xacro)
@@ -1,23 +1,48 @@
 <?xml version="1.0"?>
 <robot xmlns:xacro="http://www.ros.org/wiki/xacro" >
+  <!-- Camera sensor configuration for Gazebo Harmonic -->
   <gazebo reference="camera_link">
-  <sensor name="camera_sensor" type="camera">
-    <always_on>true</always_on>
-    <visualize>true</visualize>
-    <update_rate>30</update_rate>
-    <camera>
-      <horizontal_fov>1.047</horizontal_fov>
-      <image>
-        <width>640</width>
-        <height>480</height>
-        <format>R8G8B8</format>
-      </image>
-      <clip>
-        <near>0.1</near>
-        <far>100</far>
-      </clip>
-    </camera>
-    <topic>camera/camera_sensor</topic>
-  </sensor>
-</gazebo>
+    <sensor name="camera_sensor" type="camera">
+      <always_on>true</always_on>
+      <visualize>true</visualize>
+      <update_rate>30</update_rate>
+      <camera>
+        <horizontal_fov>1.047</horizontal_fov>
+        <image>
+          <width>640</width>
+          <height>480</height>
+          <format>R8G8B8</format>
+        </image>
+        <clip>
+          <near>0.1</near>
+          <far>100</far>
+        </clip>
+      </camera>
+    </sensor>
+  </gazebo>
+  <!-- Add material properties for all links -->
+  <gazebo reference="base_link">
+    <material>Gazebo/Grey</material>
+    <mu1>0.2</mu1>
+    <mu2>0.2</mu2>
+    <self_collide>0</self_collide>
+  </gazebo>
+  <gazebo reference="slider_link">
+    <material>Gazebo/Blue</material>
+    <mu1>0.2</mu1>
+    <mu2>0.2</mu2>
+    <self_collide>0</self_collide>
+  </gazebo>
+  <gazebo reference="arm_link">
+    <material>Gazebo/Orange</material>
+    <mu1>0.2</mu1>
+    <mu2>0.2</mu2>
+    <self_collide>0</self_collide>
+  </gazebo>
+  <gazebo reference="camera_link">
+    <material>Gazebo/White</material>
+    <mu1>0.2</mu1>
+    <mu2>0.2</mu2>
+    <self_collide>0</self_collide>
+  </gazebo>
 </robot>

File: src/vio/urdf/test_rb_1.urdf.xacro (robot description, xacro)
@@ -8,4 +8,19 @@
     <xacro:include filename="materials.xacro" />
     <xacro:include filename="gazebo.xacro" />
+    <!-- Add Gazebo plugins for proper physics and joint states -->
+    <gazebo>
+        <!-- Joint state publisher plugin for Gazebo Harmonic -->
+        <plugin name="gz::sim::systems::JointStatePublisher" filename="gz-sim-joint-state-publisher-system">
+        </plugin>
+        <!-- Pose publisher for TF -->
+        <plugin name="gz::sim::systems::PosePublisher" filename="gz-sim-pose-publisher-system">
+            <publish_link_pose>true</publish_link_pose>
+            <publish_collision_pose>false</publish_collision_pose>
+            <publish_visual_pose>false</publish_visual_pose>
+            <use_pose_vector_msg>true</use_pose_vector_msg>
+            <static_publisher>true</static_publisher>
+            <static_update_frequency>1</static_update_frequency>
+        </plugin>
+    </gazebo>
     <!-- This first link called "world" is empty -->
     <link name="world"></link>
@@ -36,11 +51,7 @@
             </geometry>
         </collision>
-        <!-- <inertial>
+        <!-- Fixed: Use actual box dimensions instead of 0,0 -->
+        <xacro:inertial_box mass="0.5" x="0.4" y="0.4" z="0.1">
             <origin xyz="0 0 0.05" rpy="0 0 0"/>
-            <mass value="12" />
-            <inertia ixx="2.26" ixy="0.0" ixz="0.0" iyy="6.26" iyz="0.0" izz="8.5" />
-        </inertial> -->
-        <xacro:inertial_box mass="0.5" x="0" y="0" z="0.1">
-            <origin xyz="0 0 0.1" rpy="0 0 0"/>
         </xacro:inertial_box>
     </link>
@@ -50,9 +61,9 @@
     <!-- - We need to specify limits for the motion -->
     <joint name="slider_joint" type="prismatic">
-        <origin xyz="-1.25 0 0.1" rpy="0 0 0"/>
+        <origin xyz="-0.25 0 0.1" rpy="0 0 0"/>
         <parent link="base_link"/>
         <child link="slider_link"/>
         <axis xyz="1 0 0"/>
-        <limit lower="0" upper="2" velocity="100" effort="100"/>
+        <limit lower="0" upper="0.5" velocity="100" effort="100"/>
     </joint>
     <!-- slider_link is the box skimming across the top of the base. Its parameters are similar to the base_link, however: -->
