Commit message: Wow, camera is no working again and drone is flying. Now I need to setup IMU

File: src/vio/urdf/_drone_gazebo.xacro (robot description, xacro)
@@ -9,7 +9,9 @@
         <plugin name="gz::sim::systems::PosePublisher" filename="gz-sim-pose-publisher-system">
             <publish_link_pose>true</publish_link_pose>
+            <publish_collision_pose>false</publish_collision_pose>
+            <publish_visual_pose>false</publish_visual_pose>
             <use_pose_vector_msg>true</use_pose_vector_msg>
             <static_publisher>true</static_publisher>
-            <static_update_frequency>10</static_update_frequency>
+            <static_update_frequency>1</static_update_frequency>
         </plugin>
         <!-- Simple velocity control that can work for basic flight -->
@@ -17,6 +19,6 @@
         </plugin>
     </gazebo>
-    <!-- Camera sensor -->
-    <gazebo reference="camera_link">
+    <!-- Camera sensor - MOVE TO BASE_LINK like working config -->
+    <gazebo reference="base_link">
         <sensor name="camera_sensor" type="camera">
             <always_on>true</always_on>
@@ -37,75 +39,53 @@
         </sensor>
     </gazebo>
-    <!-- IMU sensor -->
+    <!-- IMU sensor - keep on imu_link -->
     <gazebo reference="imu_link">
         <sensor name="imu_sensor" type="imu">
             <always_on>true</always_on>
             <update_rate>100</update_rate>
-            <imu>
-                <angular_velocity>
-                    <x>
-                        <noise type="gaussian">
-                            <mean>0.0</mean>
-                            <stddev>2e-4</stddev>
-                        </noise>
-                    </x>
-                    <y>
-                        <noise type="gaussian">
-                            <mean>0.0</mean>
-                            <stddev>2e-4</stddev>
-                        </noise>
-                    </y>
-                    <z>
-                        <noise type="gaussian">
-                            <mean>0.0</mean>
-                            <stddev>2e-4</stddev>
-                        </noise>
-                    </z>
-                </angular_velocity>
-                <linear_acceleration>
-                    <x>
-                        <noise type="gaussian">
-                            <mean>0.0</mean>
-                            <stddev>1.7e-2</stddev>
-                        </noise>
-                    </x>
-                    <y>
-                        <noise type="gaussian">
-                            <mean>0.0</mean>
-                            <stddev>1.7e-2</stddev>
-                        </noise>
-                    </y>
-                    <z>
-                        <noise type="gaussian">
-                            <mean>0.0</mean>
-                            <stddev>1.7e-2</stddev>
-                        </noise>
-                    </z>
-                </linear_acceleration>
-            </imu>
         </sensor>
     </gazebo>
-    <!-- Material properties -->
+    <!-- Add material properties for all links -->
     <gazebo reference="base_link">
         <material>Gazebo/Grey</material>
+        <mu1>0.2</mu1>
+        <mu2>0.2</mu2>
+        <self_collide>0</self_collide>
     </gazebo>
     <gazebo reference="camera_link">
         <material>Gazebo/White</material>
+        <mu1>0.2</mu1>
+        <mu2>0.2</mu2>
+        <self_collide>0</self_collide>
     </gazebo>
     <gazebo reference="imu_link">
         <material>Gazebo/Blue</material>
+        <mu1>0.2</mu1>
+        <mu2>0.2</mu2>
+        <self_collide>0</self_collide>
     </gazebo>
-    <!-- Propeller materials -->
     <gazebo reference="front_right_prop">
         <material>Gazebo/Orange</material>
+        <mu1>0.2</mu1>
+        <mu2>0.2</mu2>
+        <self_collide>0</self_collide>
     </gazebo>
     <gazebo reference="front_left_prop">
         <material>Gazebo/Orange</material>
+        <mu1>0.2</mu1>
+        <mu2>0.2</mu2>
+        <self_collide>0</self_collide>
     </gazebo>
     <gazebo reference="rear_left_prop">
         <material>Gazebo/Orange</material>
+        <mu1>0.2</mu1>
+        <mu2>0.2</mu2>
+        <self_collide>0</self_collide>
     </gazebo>
     <gazebo reference="rear_right_prop">
         <material>Gazebo/Orange</material>
+        <mu1>0.2</mu1>
+        <mu2>0.2</mu2>
+        <self_collide>0</self_collide>
     </gazebo>
 </robot>

File: src/vio/urdf/quadcopter.urdf.xacro (robot description, xacro)
@@ -130,5 +130,5 @@
         <axis xyz="0 0 1"/>
     </joint>
-    <!-- Camera gimbal -->
+    <!-- Camera gimbal - ADD COLLISION -->
     <joint name="camera_joint" type="fixed">
         <origin xyz="0.1 0 -0.05" rpy="0 0.3 0"/>
@@ -144,4 +144,5 @@
             <material name="white" />
         </visual>
+        <!-- ADD COLLISION - This is missing and needed for sensors -->
         <collision>
             <origin xyz="0 0 0" rpy="0 0 0"/>
@@ -154,5 +155,5 @@
         </xacro:inertial_box>
     </link>
-    <!-- IMU sensor link -->
+    <!-- IMU sensor link - ADD COLLISION -->
     <joint name="imu_joint" type="fixed">
         <origin xyz="0 0 0" rpy="0 0 0"/>
@@ -168,4 +169,11 @@
             <material name="blue" />
         </visual>
+        <!-- ADD COLLISION - This is missing and needed for sensors -->
+        <collision>
+            <origin xyz="0 0 0" rpy="0 0 0"/>
+            <geometry>
+                <box size="0.02 0.02 0.01" />
+            </geometry>
+        </collision>
         <xacro:inertial_box mass="0.01" x="0.02" y="0.02" z="0.01">
             <origin xyz="0 0 0" rpy="0 0 0"/>
